File: kicad/esp32c6-charger.kicad_pcb (KiCad board)
At the start: 0 parts

Commit message: moved some of the configuration to it's own file
Parts:
- added Brd1: SSD1306, Custom:128x64OLED, F.Cu at (131.4, 117.8)
- added D1: WS2812B, LED_SMD:LED_WS2812B_PLCC4_5.0x5.0mm_P3.2mm, F.Cu at (152.5, 108.3)
- added D2: Lock, LED_SMD:LED_1206_3216Metric_Pad1.42x1.75mm_HandSolder, B.Cu at (118.1, 115.1)
- added D3: Relay, LED_SMD:LED_1206_3216Metric_Pad1.42x1.75mm_HandSolder, B.Cu at (118.1, 118.9)
- added D4: Detect, LED_SMD:LED_1206_3216Metric_Pad1.42x1.75mm_HandSolder, B.Cu at (118.1, 111.3)
- added J1: Conn_01x06_Socket, TerminalBlock_Phoenix:TerminalBlock_Phoenix_MKDS-1,5-6-5.08_1x06_P5.08mm_Horizontal, B.Cu at (124.7, 95.0)
- added J2: Conn_01x03_Socket, TerminalBlock_Phoenix:TerminalBlock_Phoenix_MKDS-1,5-3-5.08_1x03_P5.08mm_Horizontal, B.Cu at (85.9, 95.2)
- added K1: G2RL-1, Relay_THT:Relay_SPDT_Omron_G2RL-1, B.Cu at (106.3, 122.8)
- added Q1: BC817, Package_TO_SOT_SMD:SOT-23-3, B.Cu at (118.0, 123.7)
- added Q2: BC817, Package_TO_SOT_SMD:SOT-23-3, B.Cu at (118.0, 128.6)
- added R1: 10k, Resistor_SMD:R_1206_3216Metric_Pad1.30x1.75mm_HandSolder, B.Cu at (125.9, 122.5)
- added R2: 10k, Resistor_SMD:R_1206_3216Metric_Pad1.30x1.75mm_HandSolder, B.Cu at (126.0, 126.2)
- added R3: 68, Resistor_SMD:R_1206_3216Metric_Pad1.30x1.75mm_HandSolder, B.Cu at (126.0, 118.9)
- added R4: 68, Resistor_SMD:R_1206_3216Metric_Pad1.30x1.75mm_HandSolder, B.Cu at (126.0, 115.1)
- added R5: 68, Resistor_SMD:R_1206_3216Metric_Pad1.30x1.75mm_HandSolder, B.Cu at (126.0, 111.3)
- added RFID1: RC522, Custom:RC522, F.Cu at (160.8, 106.2)
- added U1: XIAO-ESP32-C6, Seeed Studio XIAO Series Library:XIAO-ESP32C6-DIP, B.Cu at (141.5, 129.3)
Routing:
- net +5V: track 0.00 -> 131.2 mm
- net VCC: track 0.00 -> 103.0 mm
- net Net-(D4-K): track 0.00 -> 76.4 mm
- net Net-(D1-DIN): track 0.00 -> 49.2 mm
- net Net-(D2-K): track 0.00 -> 49.1 mm
- net Net-(J2-Pin_2): track 0.00 -> 31.7 mm
- net /MISO: track 0.00 -> 30.9 mm
- net Net-(J2-Pin_3): track 0.00 -> 29.4 mm
- net /MOSI: track 0.00 -> 27.7 mm
- net /CS: track 0.00 -> 24.3 mm
- net /SCK: track 0.00 -> 24.1 mm
- net /SDA: track 0.00 -> 21.9 mm
- net Net-(D3-K): track 0.00 -> 21.7 mm
- net /SCL: track 0.00 -> 20.3 mm
- net Net-(J2-Pin_1): track 0.00 -> 20.1 mm
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- added copper zone on B.Cu, net GND
- added copper zone on F.Cu, net GND
Other:
- board outline added: 160 x 50 mm
- copper layers 0 -> 2
- board text added: "3V3"
- board text added: "5V"
- board text added: "Detect"
- board text added: "GND"
- board text added: "Lock"
- board text added: "Make"
- board text added: "https://gertjanassies.dev/blog?category=make"
